Commit message: second commit, includes addition of readme file, removal of the test urdf file(replaced by the final xacro file)

File: nuturtle_description/urdf/diff_drive.urdf.xacro (robot description, xacro)
@@ -1,68 +1,70 @@
 <?xml version="1.0"?>
-<!-- Revolute-Revolute Manipulator -->
 <robot name="diff_drive" xmlns:xacro="http://www.ros.org/wiki/xacro">
-<xacro:property name="a" value="${load_yaml('/tsim/config/diff_params.yaml')}" />
-  <!-- Base Link -->
+<xacro:property name="yaml_file" value="$(find nuturtle_description)/config/diff_params.yaml" />
+<xacro:property name="a" value="${load_yaml(yaml_file)}"/>
+ <!-- Base Link -->
   <link name="base_link">
     <visual>
-      <origin xyz="0 0 0" rpy="0 0 0" />
+      <origin xyz="0 0 ${a['wheel_radius']}" rpy="0 0 0" />
       <geometry>
-          <box size="${a['chassis_length']} ${a['wheel_base']} ${a['chassis_thickness']} "/>
+          <box size="${a['chassis_length']} ${a['wheel_base']-a['wheel_width']} ${a['chassis_thickness']} "/>
       </geometry>
-      <material name="blue">
-        <color rgba="0 0.5 1 1"/>
+      <material name="color1">
+        <color rgba="0.1 0.3 1 1"/>
       </material>
     </visual>
   </link>
-  <!-- caster -->
-  <link name="caster">
+   <!-- Right Wheel -->
+  <link name="right_wheel">
     <visual>
-      <origin xyz="0.2 0 -0.125" rpy="0 0 0" />
+      <origin xyz="0 ${-1*a['wheel_width']/2} 0" rpy="1.570795 0 0" />
       <geometry>
-          <sphere radius="${a['wheel_radius']}"/>
+          <cylinder length="${a['wheel_width']}" radius="${a['wheel_radius']}" />
       </geometry>
-      <material name="blue">
-        <color rgba="0 0.5 1 1"/>
+      <material name="color2">
+        <color rgba="0 0 0 1"/>
       </material>
     </visual>
   </link>
-  <joint name="caster_chassis" type="floating">
+  <joint name="right_wheel_axle" type="continuous">
     <parent link="base_link"/>
-    <child link="caster"/>
-    <origin xyz="0 -0.30 0" rpy="0 0 0" />
+    <child link="right_wheel"/>
+    <origin xyz="${-1*(a['chassis_length']/2-a['wheel_radius'])} ${-1*(a['wheel_base']/2-a['wheel_width']/2)} ${a['wheel_radius']}" rpy="0 0 0" />
+    <axis xyz="0 1 0" />
   </joint>
-  <!-- Right Wheel -->
-  <link name="right_wheel">
+  <!-- left Wheel -->
+  <link name="left_wheel">
     <visual>
-      <origin xyz="0 0 0" rpy="1.570795 0 0" />
+      <origin xyz="0 ${1*a['wheel_width']/2} 0" rpy="1.570795 0 0" />
       <geometry>
           <cylinder length="${a['wheel_width']}" radius="${a['wheel_radius']}" />
       </geometry>
-      <material name="black">
-        <color rgba="0.05 0.05 0.05 1"/>
+      <material name="color3">
+        <color rgba="0.3 0.44 0.1 1"/>
       </material>
     </visual>
   </link>
-  <joint name="joint_right_wheel" type="continuous">
+  <joint name="left_wheel_axle" type="continuous">
     <parent link="base_link"/>
-    <child link="right_wheel"/>
-    <origin xyz="0 -0.30 0" rpy="0 0 0" />
+    <child link="left_wheel"/>
+    <origin xyz="${-1*(a['chassis_length']/2-a['wheel_radius'])} ${1*(a['wheel_base']/2-a['wheel_width']/2)} ${a['wheel_radius']}" rpy="0 0 0" />
     <axis xyz="0 1 0" />
   </joint>
-  <!-- Left Wheel -->
-  <link name="left_wheel">
+<!-- caster Wheel -->
+<link name="caster">
     <visual>
-      <origin xyz="0 0 0" rpy="1.570795 0 0" />
+      <origin xyz="0 0 ${-1*(a['wheel_radius']-(a['chassis_thickness']/2))/2}" rpy="0 0 0" />
       <geometry>
-          <cylinder length="${a['wheel_width']}" radius="${a['wheel_radius']}" />
+          <sphere radius="${(a['wheel_radius']-(a['chassis_thickness']/2))/2}"/>
       </geometry>
-      <material name="black"/>
+      <material name="color4">
+        <color rgba="0.8 0.12 1 1"/>
+      </material>
     </visual>
   </link>
-  <joint name="joint_left_wheel" type="continuous">
+  <joint name="caster_chassis" type="fixed">
     <parent link="base_link"/>
-    <child link="left_wheel"/>
-    <origin xyz="0 0.30 0" rpy="0 0 0" />
-    <axis xyz="0 1 0" />
+    <child link="caster"/>
+    <origin xyz="${a['chassis_length']/2-(a['wheel_radius']-(a['chassis_thickness']/2))/2} 0 ${-1*a['chassis_thickness']/2 + a['wheel_radius']}" />
   </joint>
 </robot>

Commit message: changed base link reference frame which was wrong. added description to launch file

File: nuturtle_description/urdf/diff_drive.urdf.xacro (robot description, xacro)
@@ -6,5 +6,5 @@
   <link name="base_link">
     <visual>
-      <origin xyz="0 0 ${a['wheel_radius']}" rpy="0 0 0" />
+      <origin xyz="${a['chassis_length']/2 - a['wheel_radius']} 0 ${a['wheel_radius']}" rpy="0 0 0" />
       <geometry>
           <box size="${a['chassis_length']} ${a['wheel_base']-a['wheel_width']} ${a['chassis_thickness']} "/>
@@ -30,5 +30,5 @@
     <parent link="base_link"/>
     <child link="right_wheel"/>
-    <origin xyz="${-1*(a['chassis_length']/2-a['wheel_radius'])} ${-1*(a['wheel_base']/2-a['wheel_width']/2)} ${a['wheel_radius']}" rpy="0 0 0" />
+    <origin xyz="0 ${-1*(a['wheel_base']/2-a['wheel_width']/2)} ${a['wheel_radius']}" rpy="0 0 0" />
     <axis xyz="0 1 0" />
   </joint>
@@ -48,5 +48,5 @@
     <parent link="base_link"/>
     <child link="left_wheel"/>
-    <origin xyz="${-1*(a['chassis_length']/2-a['wheel_radius'])} ${1*(a['wheel_base']/2-a['wheel_width']/2)} ${a['wheel_radius']}" rpy="0 0 0" />
+    <origin xyz="0 ${1*(a['wheel_base']/2-a['wheel_width']/2)} ${a['wheel_radius']}" rpy="0 0 0" />
     <axis xyz="0 1 0" />
   </joint>
@@ -66,5 +66,5 @@
     <parent link="base_link"/>
     <child link="caster"/>
-    <origin xyz="${a['chassis_length']/2-(a['wheel_radius']-(a['chassis_thickness']/2))/2} 0 ${-1*a['chassis_thickness']/2 + a['wheel_radius']}" />
+    <origin xyz="${a['chassis_length']-(a['wheel_radius']-(a['chassis_thickness']/2))/2 - a['wheel_radius']} 0 ${-1*a['chassis_thickness']/2 + a['wheel_radius']}" />
   </joint>
 </robot>

Commit message: hw1 commit 2

File: nuturtle_description/urdf/diff_drive.urdf.xacro (robot description, xacro)
@@ -63,8 +63,9 @@
     </visual>
   </link>
-  <joint name="caster_chassis" type="fixed">
+  <joint name="caster_chassis" type="continuous">
     <parent link="base_link"/>
     <child link="caster"/>
     <origin xyz="${a['chassis_length']-(a['wheel_radius']-(a['chassis_thickness']/2))/2 - a['wheel_radius']} 0 ${-1*a['chassis_thickness']/2 + a['wheel_radius']}" />
+    <axis xyz = '1 1 1'/>
   </joint>
 </robot>

Commit message: hw1_almost final

File: nuturtle_description/urdf/diff_drive.urdf.xacro (robot description, xacro)
@@ -67,5 +67,5 @@
     <child link="caster"/>
     <origin xyz="${a['chassis_length']-(a['wheel_radius']-(a['chassis_thickness']/2))/2 - a['wheel_radius']} 0 ${-1*a['chassis_thickness']/2 + a['wheel_radius']}" />
-    <axis xyz = '1 1 1'/>
+    <axis xyz = '1 1 0'/>
   </joint>
 </robot>

Commit message: pentagon running on bot

File: nuturtle_description/urdf/diff_drive.urdf.xacro (robot description, xacro)
@@ -63,5 +63,5 @@
     </visual>
   </link>
-  <joint name="caster_chassis" type="continuous">
+  <joint name="caster_chassis" type="fixed">
     <parent link="base_link"/>
     <child link="caster"/>

Commit message: finished hw. to add comments

File: nuturtle_description/urdf/diff_drive.urdf.xacro (robot description, xacro)
@@ -6,5 +6,5 @@
   <link name="base_link">
     <visual>
-      <origin xyz="${a['chassis_length']/2 - a['wheel_radius']} 0 ${a['wheel_radius']}" rpy="0 0 0" />
+      <origin xyz="${a['chassis_length']/2 - a['wheel_radius']} 0 ${a['chassis_thickness']/2 + a['wheel_radius']}" rpy="0 0 0" />
       <geometry>
           <box size="${a['chassis_length']} ${a['wheel_base']-a['wheel_width']} ${a['chassis_thickness']} "/>
@@ -54,7 +54,7 @@
 <link name="caster">
     <visual>
-      <origin xyz="0 0 ${-1*(a['wheel_radius']-(a['chassis_thickness']/2))/2}" rpy="0 0 0" />
+      <origin xyz="0 0 0" rpy="0 0 0" />
       <geometry>
-          <sphere radius="${(a['wheel_radius']-(a['chassis_thickness']/2))/2}"/>
+          <sphere radius="${a['wheel_radius'] /2 }"/>
       </geometry>
       <material name="color4">
@@ -66,5 +66,5 @@
     <parent link="base_link"/>
     <child link="caster"/>
-    <origin xyz="${a['chassis_length']-(a['wheel_radius']-(a['chassis_thickness']/2))/2 - a['wheel_radius']} 0 ${-1*a['chassis_thickness']/2 + a['wheel_radius']}" />
+    <origin xyz="${a['chassis_length']-a['wheel_radius']- 0.005} 0 ${a['wheel_radius']/2}" />
     <axis xyz = '1 1 0'/>
   </joint>

Commit message: finished plugin

File: nuturtle_description/urdf/diff_drive.urdf.xacro (robot description, xacro)
@@ -3,8 +3,13 @@
 <xacro:property name="yaml_file" value="$(find nuturtle_description)/config/diff_params.yaml" />
 <xacro:property name="a" value="${load_yaml(yaml_file)}"/>
- <!-- Base Link -->
-  <link name="base_link">
+  <link name="base_link"/>
+  <joint name="base_joint" type="fixed">
+    <parent link="body_link"/>
+    <child link="base_link"/>
+    <origin xyz="0.0 0.0 0.0" rpy="0 0 0"/>
+  </joint>
+  <link name="body_link">
     <visual>
-      <origin xyz="${a['chassis_length']/2 - a['wheel_radius']} 0 ${a['chassis_thickness']/2 + a['wheel_radius']}" rpy="0 0 0" />
+      <origin xyz="${a['chassis_length']/2 - a['wheel_radius']} 0 ${a['chassis_thickness']/2 + a['wheel_axle_offset']}" rpy="0 0 0" />
       <geometry>
           <box size="${a['chassis_length']} ${a['wheel_base']-a['wheel_width']} ${a['chassis_thickness']} "/>
@@ -14,5 +19,17 @@
       </material>
     </visual>
-  </link>
+    <collision>
+      <origin xyz="${a['chassis_length']/2 - a['wheel_radius']} 0 ${a['chassis_thickness']/2 + a['wheel_radius']}" rpy="0 0 0" />
+      <geometry>
+         <box size="${a['chassis_length']} ${a['wheel_base']-a['wheel_width']} ${a['chassis_thickness']} "/>
+      </geometry>
+    </collision>
+    <inertial>
+      <mass value="0.94"/>
+      <inertia ixx="0.1" ixy="0.0" ixz="0.0"
+               iyy="0.1" iyz="0.0"
+               izz="0.1" />
+     </inertial>
+</link>
    <!-- Right Wheel -->
   <link name="right_wheel">
@@ -26,7 +43,19 @@
       </material>
     </visual>
+    <collision>
+      <origin xyz="0 ${-1*a['wheel_width']/2} 0" rpy="1.570795 0 0" />
+      <geometry>
+      <cylinder length="${a['wheel_width']}" radius="${a['wheel_radius']}" />
+      </geometry>
+    </collision>
+    <inertial>
+      <mass value="0.03"/>
+      <inertia ixx="1.1175580e-05" ixy="-4.2369783e-11" ixz="-5.9381719e-09"
+               iyy="1.1192413e-05" iyz="-1.4400107e-11"
+               izz="2.0712558e-05" />
+    </inertial>
   </link>
   <joint name="right_wheel_axle" type="continuous">
-    <parent link="base_link"/>
+    <parent link="body_link"/>
     <child link="right_wheel"/>
     <origin xyz="0 ${-1*(a['wheel_base']/2-a['wheel_width']/2)} ${a['wheel_radius']}" rpy="0 0 0" />
@@ -44,7 +73,19 @@
       </material>
     </visual>
+    <collision>
+      <origin xyz="0 ${1*a['wheel_width']/2} 0" rpy="1.570795 0 0" />
+      <geometry>
+      <cylinder length="${a['wheel_width']}" radius="${a['wheel_radius']}" />
+      </geometry>
+    </collision>
+    <inertial>
+      <mass value="0.03"/>
+     <inertia ixx="1.1175580e-05" ixy="-4.2369783e-11" ixz="-5.9381719e-09"
+               iyy="1.1192413e-05" iyz="-1.4400107e-11"
+               izz="2.0712558e-05" />
+    </inertial>
   </link>
   <joint name="left_wheel_axle" type="continuous">
-    <parent link="base_link"/>
+    <parent link="body_link"/>
     <child link="left_wheel"/>
     <origin xyz="0 ${1*(a['wheel_base']/2-a['wheel_width']/2)} ${a['wheel_radius']}" rpy="0 0 0" />
@@ -62,7 +103,13 @@
       </material>
     </visual>
+    <collision>
+      <origin xyz="0 0 0" rpy="0 0 0" />
+      <geometry>
+      <sphere radius="${a['wheel_radius'] /2 }"/>
+      </geometry>
+    </collision>
   </link>
   <joint name="caster_chassis" type="fixed">
-    <parent link="base_link"/>
+    <parent link="body_link"/>
     <child link="caster"/>
     <origin xyz="${a['chassis_length']-a['wheel_radius']- 0.005} 0 ${a['wheel_radius']/2}" />

Commit message: working on landmark detection

File: nuturtle_description/urdf/diff_drive.urdf.xacro (robot description, xacro)
@@ -5,6 +5,6 @@
   <link name="base_link"/>
   <joint name="base_joint" type="fixed">
-    <parent link="body_link"/>
-    <child link="base_link"/>
+    <parent link="base_link"/>
+    <child link="body_link"/>
     <origin xyz="0.0 0.0 0.0" rpy="0 0 0"/>
   </joint>
@@ -32,4 +32,21 @@
      </inertial>
 </link>
+<link name = "base_scan">
+    <visual>
+      <origin xyz="0 0 0" rpy="0 0 0" />
+      <geometry>
+          <cylinder length="0.005" radius="${(a['wheel_base']-a['wheel_width'])/2}" />
+      </geometry>
+      <material name="color2">
+        <color rgba="0 0 0 1"/>
+      </material>
+    </visual>
+</link>
+   <joint name="scan_joint" type="fixed">
+    <parent link="body_link"/>
+    <child link="base_scan"/>
+    <origin xyz="${a['chassis_length']/2 - a['wheel_radius']} 0 ${a['chassis_thickness'] + a['wheel_axle_offset']}" rpy="0 0 0" />
+    <axis xyz="0 1 0" />
+  </joint>
    <!-- Right Wheel -->
   <link name="right_wheel">

File: nuturtle_gazebo/urdf/diff_drive.gazebo.xacro (robot description, xacro)
@@ -4,6 +4,6 @@
   <gazebo>
     <plugin name="turtle_drive_plugin" filename="libnuturtle_gazebo_plugin.so">
-    <sensor_data_topic>sensor_data</sensor_data_topic>
-    <wheel_cmd_topic>wheel_cmd</wheel_cmd_topic>
+    <sensor_data_topic>/sensor_data</sensor_data_topic>
+    <wheel_cmd_topic>/wheel_cmd</wheel_cmd_topic>
     <left_wheel_joint>left_wheel_axle</left_wheel_joint>
     <right_wheel_joint>right_wheel_axle</right_wheel_joint>
@@ -42,3 +42,35 @@
     <material>Gazebo/FlatBlack</material>
   </gazebo>
+<gazebo reference="base_scan">
+  <material>Gazebo/FlatBlack</material>
+  <sensor type="ray" name="lds_lfcd_sensor">
+    <pose>0 0 0 0 0 0</pose>
+    <visualize>true</visualize>
+    <update_rate>5</update_rate>
+    <ray>
+      <scan>
+        <horizontal>
+          <samples>360</samples>
+          <resolution>1</resolution>
+          <min_angle>0.0</min_angle>
+          <max_angle>6.28319</max_angle>
+        </horizontal>
+      </scan>
+      <range>
+        <min>0.120</min>
+        <max>3.5</max>
+        <resolution>0.015</resolution>
+      </range>
+      <noise>
+        <type>gaussian</type>
+        <mean>0.0</mean>
+        <stddev>0.01</stddev>
+      </noise>
+    </ray>
+    <plugin name="gazebo_ros_lds_lfcd_controller" filename="libgazebo_ros_laser.so">
+      <topicName>scan</topicName>
+      <frameName>base_scan</frameName>
+    </plugin>
+  </sensor>
+</gazebo>
 </robot>

Commit message: working on slam with known data associtaiton

File: nuturtle_description/urdf/diff_drive.urdf.xacro (robot description, xacro)
@@ -3,4 +3,13 @@
 <xacro:property name="yaml_file" value="$(find nuturtle_description)/config/diff_params.yaml" />
 <xacro:property name="a" value="${load_yaml(yaml_file)}"/>
+<xacro:property name="l" value="${a['chassis_length']}" />
+<xacro:property name="w" value="${a['wheel_base']}" />
+<xacro:property name="h" value="${a['chassis_thickness']}" />
+<xacro:property name="w_off" value="${a['wheel_axle_offset']}" />
+<xacro:property name="r" value="${a['wheel_radius']}" />
+<xacro:property name="wid" value="${a['wheel_width']}" />
+<xacro:property name="r_o" value="${(r - w_off)/2}" />
+<xacro:property name="mass_c" value="${a['chassis_mass']}" />
+<xacro:property name="mass_w" value="${a['wheel_mass']}" />
   <link name="base_link"/>
   <joint name="base_joint" type="fixed">
@@ -11,5 +20,5 @@
   <link name="body_link">
     <visual>
-      <origin xyz="${a['chassis_length']/2 - a['wheel_radius']} 0 ${a['chassis_thickness']/2 + a['wheel_axle_offset']}" rpy="0 0 0" />
+      <origin xyz="${a['chassis_length']/2 - a['wheel_radius']} 0 ${a['chassis_thickness']/2 +a['wheel_radius']- a['wheel_axle_offset']}" rpy="0 0 0" />
       <geometry>
           <box size="${a['chassis_length']} ${a['wheel_base']-a['wheel_width']} ${a['chassis_thickness']} "/>
@@ -20,5 +29,5 @@
     </visual>
     <collision>
-      <origin xyz="${a['chassis_length']/2 - a['wheel_radius']} 0 ${a['chassis_thickness']/2 + a['wheel_radius']}" rpy="0 0 0" />
+      <origin xyz="${a['chassis_length']/2 - a['wheel_radius']} 0 ${a['chassis_thickness']/2 + a['wheel_radius']- a['wheel_axle_offset']}" rpy="0 0 0" />
       <geometry>
          <box size="${a['chassis_length']} ${a['wheel_base']-a['wheel_width']} ${a['chassis_thickness']} "/>
@@ -26,8 +35,8 @@
     </collision>
     <inertial>
-      <mass value="0.94"/>
-      <inertia ixx="0.1" ixy="0.0" ixz="0.0"
-               iyy="0.1" iyz="0.0"
-               izz="0.1" />
+      <mass value="${mass_c}"/>
+      <inertia  ixx="${mass_c * ( (h*h) + ((w-wid)*(w-wid)) ) / 12.0}" ixy="0" ixz="0"
+              iyy="${mass_c * ( (l*l) + ((w-wid)*(w-wid)) ) / 12.0}" iyz="0"
+              izz="${mass_c * ((h*h) + (l*l)) / 12.0}"/> />
      </inertial>
 </link>
@@ -36,5 +45,5 @@
       <origin xyz="0 0 0" rpy="0 0 0" />
       <geometry>
-          <cylinder length="0.005" radius="${(a['wheel_base']-a['wheel_width'])/2}" />
+          <cylinder length="0.039" radius="${(a['wheel_base']-a['wheel_width'])/4}" />
       </geometry>
       <material name="color2">
@@ -46,5 +55,5 @@
     <parent link="body_link"/>
     <child link="base_scan"/>
-    <origin xyz="${a['chassis_length']/2 - a['wheel_radius']} 0 ${a['chassis_thickness'] + a['wheel_axle_offset']}" rpy="0 0 0" />
+    <origin xyz="${a['chassis_length']/2 - a['wheel_radius']} 0 ${a['chassis_thickness'] +  a['wheel_radius']- a['wheel_axle_offset'] + 0.0195}" rpy="0 0 0" />
     <axis xyz="0 1 0" />
   </joint>
@@ -67,8 +76,8 @@
     </collision>
     <inertial>
-      <mass value="0.03"/>
-      <inertia ixx="1.1175580e-05" ixy="-4.2369783e-11" ixz="-5.9381719e-09"
-               iyy="1.1192413e-05" iyz="-1.4400107e-11"
-               izz="2.0712558e-05" />
+      <mass value="${mass_w}"/>
+      <inertia  ixx="${mass_w * ((3*r*r)+ (wid*wid)) / 12.0}"
+              iyy="${mass_w * ((3*r*r)+ (wid*wid)) / 12.0}" iyz="0"
+              izz="${0.5 * mass_w * (r*r)}" ixy="0" ixz="0"/>
     </inertial>
   </link>
@@ -97,9 +106,9 @@
     </collision>
     <inertial>
-      <mass value="0.03"/>
-     <inertia ixx="1.1175580e-05" ixy="-4.2369783e-11" ixz="-5.9381719e-09"
-               iyy="1.1192413e-05" iyz="-1.4400107e-11"
-               izz="2.0712558e-05" />
-    </inertial>
+      <mass value="${mass_w}"/>
+   <inertia  ixx="${mass_w * ((3*r*r)+ (wid*wid)) / 12.0}"
+              iyy="${mass_w * ((3*r*r)+ (wid*wid)) / 12.0}" iyz="0"
+              izz="${0.5 * mass_w * (r*r)}" ixy="0" ixz="0"/>
+   </inertial>
   </link>
   <joint name="left_wheel_axle" type="continuous">

File: nuturtle_gazebo/urdf/diff_drive.gazebo.xacro (robot description, xacro)
@@ -8,5 +8,5 @@
     <left_wheel_joint>left_wheel_axle</left_wheel_joint>
     <right_wheel_joint>right_wheel_axle</right_wheel_joint>
-    <sensor_frequency>250</sensor_frequency>
+    <sensor_frequency>100</sensor_frequency>
     </plugin>
   </gazebo>
@@ -16,24 +16,31 @@
   <gazebo reference="body_link">
     <material>Gazebo/DarkGrey</material>
+    <minDepth>0.001</minDepth>
   </gazebo>
   <gazebo reference="left_wheel">
-    <mu1>0.1</mu1>
-    <mu2>0.1</mu2>
+    <mu1>0.8</mu1>
+    <mu2>0.8</mu2>
     <minDepth>0.001</minDepth>
     <maxVel>0.1</maxVel>
     <fdir1>1 0 0</fdir1>
+    <kp>500000</kp>
+    <kd>10</kd>
+    <dampingFactor> 1 </dampingFactor>
     <material>Gazebo/FlatBlack</material>
   </gazebo>
   <gazebo reference="right_wheel">
-    <mu1>0.1</mu1>
-    <mu2>0.1</mu2>
+    <mu1>0.8</mu1>
+    <mu2>0.8</mu2>
     <minDepth>0.001</minDepth>
     <maxVel>0.1</maxVel>
     <fdir1>1 0 0</fdir1>
+    <kp>500000</kp>
+    <kd>10</kd>
+    <dampingFactor> 1 </dampingFactor>
     <material>Gazebo/FlatBlack</material>
   </gazebo>
-  <gazebo reference="caster_back_link">
-    <mu1>0.1</mu1>
-    <mu2>0.1</mu2>
+  <gazebo reference="caster">
+    <mu1>0.02</mu1>
+    <mu2>0.02</mu2>
     <minDepth>0.001</minDepth>
     <maxVel>1.0</maxVel>
@@ -65,5 +72,5 @@
         <type>gaussian</type>
         <mean>0.0</mean>
-        <stddev>0.01</stddev>
+        <stddev>0</stddev>
       </noise>
     </ray>
