Commit message: slam seems to work with known data association

File: nuturtle_description/urdf/diff_drive.urdf.xacro (robot description, xacro)
@@ -9,18 +9,18 @@
 <xacro:property name="r" value="${a['wheel_radius']}" />
 <xacro:property name="wid" value="${a['wheel_width']}" />
-<xacro:property name="r_o" value="${(r - w_off)/2}" />
 <xacro:property name="mass_c" value="${a['chassis_mass']}" />
 <xacro:property name="mass_w" value="${a['wheel_mass']}" />
+<xacro:property name="caster_rad" value="${(r-w_off)/2}" />
   <link name="base_link"/>
   <joint name="base_joint" type="fixed">
     <parent link="base_link"/>
     <child link="body_link"/>
-    <origin xyz="0.0 0.0 0.0" rpy="0 0 0"/>
+    <origin xyz="${l/2 - r} 0.0 ${h/2 +r- w_off}" rpy="0 0 0"/>
   </joint>
   <link name="body_link">
     <visual>
-      <origin xyz="${a['chassis_length']/2 - a['wheel_radius']} 0 ${a['chassis_thickness']/2 +a['wheel_radius']- a['wheel_axle_offset']}" rpy="0 0 0" />
+      <origin xyz="0 0 0" rpy="0 0 0" />
       <geometry>
-          <box size="${a['chassis_length']} ${a['wheel_base']-a['wheel_width']} ${a['chassis_thickness']} "/>
+          <box size="${l} ${w-wid} ${h} "/>
       </geometry>
       <material name="color1">
@@ -29,31 +29,22 @@
     </visual>
     <collision>
-      <origin xyz="${a['chassis_length']/2 - a['wheel_radius']} 0 ${a['chassis_thickness']/2 + a['wheel_radius']- a['wheel_axle_offset']}" rpy="0 0 0" />
+      <origin xyz="${l/2 - r} 0 ${h/2 + r- w_off}" rpy="0 0 0" />
       <geometry>
-         <box size="${a['chassis_length']} ${a['wheel_base']-a['wheel_width']} ${a['chassis_thickness']} "/>
+         <box size="${l} ${w-wid} ${h} "/>
       </geometry>
     </collision>
     <inertial>
       <mass value="${mass_c}"/>
-      <inertia  ixx="${mass_c * ( (h*h) + ((w-wid)*(w-wid)) ) / 12.0}" ixy="0" ixz="0"
-              iyy="${mass_c * ( (l*l) + ((w-wid)*(w-wid)) ) / 12.0}" iyz="0"
-              izz="${mass_c * ((h*h) + (l*l)) / 12.0}"/> />
+      <inertia  ixx="${mass_c * ((h*h)+ (w-wid)*(w-wid))/12}" ixy="0" ixz="0"
+              iyy="${mass_c * ((w-wid)*(w-wid) + l*l)/12}" iyz="0"
+              izz="${mass_c * (h*h + l*l)/12 }"/> />
      </inertial>
 </link>
 <link name = "base_scan">
-    <visual>
-      <origin xyz="0 0 0" rpy="0 0 0" />
-      <geometry>
-          <cylinder length="0.039" radius="${(a['wheel_base']-a['wheel_width'])/4}" />
-      </geometry>
-      <material name="color2">
-        <color rgba="0 0 0 1"/>
-      </material>
-    </visual>
-</link>
+  </link>
    <joint name="scan_joint" type="fixed">
     <parent link="body_link"/>
     <child link="base_scan"/>
-    <origin xyz="${a['chassis_length']/2 - a['wheel_radius']} 0 ${a['chassis_thickness'] +  a['wheel_radius']- a['wheel_axle_offset'] + 0.0195}" rpy="0 0 0" />
+    <origin xyz="0 0 ${h/2 +0.01}" rpy="0 0 0" />
     <axis xyz="0 1 0" />
   </joint>
@@ -61,7 +52,7 @@
   <link name="right_wheel">
     <visual>
-      <origin xyz="0 ${-1*a['wheel_width']/2} 0" rpy="1.570795 0 0" />
+      <origin xyz="0 ${-1*wid/2} 0" rpy="1.570795 0 0" />
       <geometry>
-          <cylinder length="${a['wheel_width']}" radius="${a['wheel_radius']}" />
+          <cylinder length="${wid}" radius="${r}" />
       </geometry>
       <material name="color2">
@@ -70,7 +61,7 @@
     </visual>
     <collision>
-      <origin xyz="0 ${-1*a['wheel_width']/2} 0" rpy="1.570795 0 0" />
+      <origin xyz="0 ${-1*wid/2} 0" rpy="1.570795 0 0" />
       <geometry>
-      <cylinder length="${a['wheel_width']}" radius="${a['wheel_radius']}" />
+      <cylinder length="${wid}" radius="${r}" />
       </geometry>
     </collision>
@@ -85,5 +76,5 @@
     <parent link="body_link"/>
     <child link="right_wheel"/>
-    <origin xyz="0 ${-1*(a['wheel_base']/2-a['wheel_width']/2)} ${a['wheel_radius']}" rpy="0 0 0" />
+    <origin xyz="${-l/2 + r} ${-1*(w/2-wid/2)} ${-h/2 + w_off}" rpy="0 0 0" />
     <axis xyz="0 1 0" />
   </joint>
@@ -91,7 +82,7 @@
   <link name="left_wheel">
     <visual>
-      <origin xyz="0 ${1*a['wheel_width']/2} 0" rpy="1.570795 0 0" />
+      <origin xyz="0 ${1*wid/2} 0" rpy="1.570795 0 0" />
       <geometry>
-          <cylinder length="${a['wheel_width']}" radius="${a['wheel_radius']}" />
+          <cylinder length="${wid}" radius="${r}" />
       </geometry>
       <material name="color3">
@@ -100,7 +91,7 @@
     </visual>
     <collision>
-      <origin xyz="0 ${1*a['wheel_width']/2} 0" rpy="1.570795 0 0" />
+      <origin xyz="0 ${1*wid/2} 0" rpy="1.570795 0 0" />
       <geometry>
-      <cylinder length="${a['wheel_width']}" radius="${a['wheel_radius']}" />
+      <cylinder length="${wid}" radius="${r}" />
       </geometry>
     </collision>
@@ -115,5 +106,5 @@
     <parent link="body_link"/>
     <child link="left_wheel"/>
-    <origin xyz="0 ${1*(a['wheel_base']/2-a['wheel_width']/2)} ${a['wheel_radius']}" rpy="0 0 0" />
+    <origin xyz="${-l/2 + r} ${1*(w/2-wid/2)} ${-h/2 + w_off}" rpy="0 0 0" />
     <axis xyz="0 1 0" />
   </joint>
@@ -123,5 +114,5 @@
       <origin xyz="0 0 0" rpy="0 0 0" />
       <geometry>
-          <sphere radius="${a['wheel_radius'] /2 }"/>
+          <sphere radius="${caster_rad }"/>
       </geometry>
       <material name="color4">
@@ -132,5 +123,5 @@
       <origin xyz="0 0 0" rpy="0 0 0" />
       <geometry>
-      <sphere radius="${a['wheel_radius'] /2 }"/>
+      <sphere radius="${caster_rad}"/>
       </geometry>
     </collision>
@@ -139,6 +130,6 @@
     <parent link="body_link"/>
     <child link="caster"/>
-    <origin xyz="${a['chassis_length']-a['wheel_radius']- 0.005} 0 ${a['wheel_radius']/2}" />
-    <axis xyz = '1 1 0'/>
+    <origin xyz="${l/2 - caster_rad} 0 ${-h/2 - caster_rad}" />
+    <axis xyz = '1 1 1'/>
   </joint>
 </robot>

File: nuturtle_gazebo/urdf/diff_drive.gazebo.xacro (robot description, xacro)
@@ -41,6 +41,6 @@
   </gazebo>
   <gazebo reference="caster">
-    <mu1>0.02</mu1>
-    <mu2>0.02</mu2>
+    <mu1>0.2</mu1>
+    <mu2>0.2</mu2>
     <minDepth>0.001</minDepth>
     <maxVel>1.0</maxVel>
@@ -72,5 +72,5 @@
         <type>gaussian</type>
         <mean>0.0</mean>
-        <stddev>0</stddev>
+        <stddev>0.01</stddev>
       </noise>
     </ray>

Commit message: made changes in launch file to better suit final structure

File: nuturtle_description/urdf/diff_drive.urdf.xacro (robot description, xacro)
@@ -16,9 +16,9 @@
     <parent link="base_link"/>
     <child link="body_link"/>
-    <origin xyz="${l/2 - r} 0.0 ${h/2 +r- w_off}" rpy="0 0 0"/>
+     <origin xyz="${l/2 - r} 0.0 ${h/2 +r- w_off}" rpy="0 0 0"/>
   </joint>
   <link name="body_link">
     <visual>
-      <origin xyz="0 0 0" rpy="0 0 0" />
+     <origin xyz="0 0 0" rpy="0 0 0" />
       <geometry>
           <box size="${l} ${w-wid} ${h} "/>
@@ -34,17 +34,26 @@
       </geometry>
     </collision>
-    <inertial>
+     <inertial>
       <mass value="${mass_c}"/>
-      <inertia  ixx="${mass_c * ((h*h)+ (w-wid)*(w-wid))/12}" ixy="0" ixz="0"
+     <inertia  ixx="${mass_c * ((h*h)+ (w-wid)*(w-wid))/12}" ixy="0" ixz="0"
               iyy="${mass_c * ((w-wid)*(w-wid) + l*l)/12}" iyz="0"
               izz="${mass_c * (h*h + l*l)/12 }"/> />
      </inertial>
 </link>
-<link name = "base_scan">
-  </link>
+<link name ="base_scan">
+    <visual>
+      <origin xyz="0 0 0" rpy="0 0 0" />
+      <geometry>
+          <cylinder length="0.02" radius="${(w-wid)/4}" />
+      </geometry>
+      <material name="color2">
+        <color rgba="0 0 0 1"/>
+      </material>
+    </visual>
+</link>
    <joint name="scan_joint" type="fixed">
     <parent link="body_link"/>
     <child link="base_scan"/>
-    <origin xyz="0 0 ${h/2 +0.01}" rpy="0 0 0" />
+    <origin xyz="${l/4} 0 ${h/2 + 0.02/2}" rpy="0 0 0" />
     <axis xyz="0 1 0" />
   </joint>
@@ -52,5 +61,5 @@
   <link name="right_wheel">
     <visual>
-      <origin xyz="0 ${-1*wid/2} 0" rpy="1.570795 0 0" />
+       <origin xyz="0 ${-1*wid/2} 0" rpy="1.570795 0 0" />
       <geometry>
           <cylinder length="${wid}" radius="${r}" />
@@ -76,5 +85,5 @@
     <parent link="body_link"/>
     <child link="right_wheel"/>
-    <origin xyz="${-l/2 + r} ${-1*(w/2-wid/2)} ${-h/2 + w_off}" rpy="0 0 0" />
+   <origin xyz="${-l/2 + r} ${-1*(w/2-wid/2)} ${-h/2 + w_off}" rpy="0 0 0" />
     <axis xyz="0 1 0" />
   </joint>
@@ -82,5 +91,5 @@
   <link name="left_wheel">
     <visual>
-      <origin xyz="0 ${1*wid/2} 0" rpy="1.570795 0 0" />
+   <origin xyz="0 ${1*wid/2} 0" rpy="1.570795 0 0" />
       <geometry>
           <cylinder length="${wid}" radius="${r}" />
@@ -98,13 +107,13 @@
     <inertial>
       <mass value="${mass_w}"/>
-   <inertia  ixx="${mass_w * ((3*r*r)+ (wid*wid)) / 12.0}"
+     <inertia  ixx="${mass_w * ((3*r*r)+ (wid*wid)) / 12.0}"
               iyy="${mass_w * ((3*r*r)+ (wid*wid)) / 12.0}" iyz="0"
               izz="${0.5 * mass_w * (r*r)}" ixy="0" ixz="0"/>
-   </inertial>
+    </inertial>
   </link>
   <joint name="left_wheel_axle" type="continuous">
     <parent link="body_link"/>
     <child link="left_wheel"/>
-    <origin xyz="${-l/2 + r} ${1*(w/2-wid/2)} ${-h/2 + w_off}" rpy="0 0 0" />
+   <origin xyz="${-l/2 + r} ${1*(w/2-wid/2)} ${-h/2 + w_off}" rpy="0 0 0" />
     <axis xyz="0 1 0" />
   </joint>
@@ -126,9 +135,9 @@
       </geometry>
     </collision>
-  </link>
+ </link>
   <joint name="caster_chassis" type="fixed">
     <parent link="body_link"/>
     <child link="caster"/>
-    <origin xyz="${l/2 - caster_rad} 0 ${-h/2 - caster_rad}" />
+  <origin xyz="${l/2 - caster_rad} 0 ${-h/2 - caster_rad}" />
     <axis xyz = '1 1 1'/>
   </joint>

Commit message: made changes in gazebo props as the bot was slipping a lot corrected mistakes in ekf update step

File: nuturtle_description/urdf/diff_drive.urdf.xacro (robot description, xacro)
@@ -42,18 +42,9 @@
 </link>
 <link name ="base_scan">
-    <visual>
-      <origin xyz="0 0 0" rpy="0 0 0" />
-      <geometry>
-          <cylinder length="0.02" radius="${(w-wid)/4}" />
-      </geometry>
-      <material name="color2">
-        <color rgba="0 0 0 1"/>
-      </material>
-    </visual>
 </link>
    <joint name="scan_joint" type="fixed">
-    <parent link="body_link"/>
+    <parent link="base_link"/>
     <child link="base_scan"/>
-    <origin xyz="${l/4} 0 ${h/2 + 0.02/2}" rpy="0 0 0" />
+    <origin xyz="0 0 ${h/2 + 0.03/2}" rpy="0 0 0" />
     <axis xyz="0 1 0" />
   </joint>

File: nuturtle_gazebo/urdf/diff_drive.gazebo.xacro (robot description, xacro)
@@ -19,21 +19,20 @@
   </gazebo>
   <gazebo reference="left_wheel">
-    <mu1>0.8</mu1>
-    <mu2>0.8</mu2>
+   <mu1>500</mu1>
+    <mu2>500</mu2>
     <minDepth>0.001</minDepth>
     <maxVel>0.1</maxVel>
     <fdir1>1 0 0</fdir1>
-    <kp>500000</kp>
+    <kp>800000</kp>
     <kd>10</kd>
     <dampingFactor> 1 </dampingFactor>
-    <material>Gazebo/FlatBlack</material>
   </gazebo>
   <gazebo reference="right_wheel">
-    <mu1>0.8</mu1>
-    <mu2>0.8</mu2>
+    <mu1>100</mu1>
+    <mu2>100</mu2>
     <minDepth>0.001</minDepth>
     <maxVel>0.1</maxVel>
     <fdir1>1 0 0</fdir1>
-    <kp>500000</kp>
+    <kp>850000</kp>
     <kd>10</kd>
     <dampingFactor> 1 </dampingFactor>
@@ -41,6 +40,6 @@
   </gazebo>
   <gazebo reference="caster">
-    <mu1>0.2</mu1>
-    <mu2>0.2</mu2>
+    <mu1>0.0001</mu1>
+    <mu2>0.0001</mu2>
     <minDepth>0.001</minDepth>
     <maxVel>1.0</maxVel>
